Commit message: added laser scan and navigation pkg

File: steer_bot_description/urdf/steer_bot.urdf.xacro (robot description, xacro)
@@ -134,7 +134,62 @@
     <origin xyz="${-base_length/2+axle_offset} ${+base_width/2+axle_offset} 0" rpy="${-90 * deg_to_rad} 0 0"/>
   </xacro:rear_wheel_lr>
+<!--   <joint name="laser_sensor_joint" type="fixed">
+      <origin xyz="0.2 0.0 ${base_height}" rpy="0 0 0"/>
+      <parent link="base_link"/>
+      <child link="laser_sensor_link"/>
+  </joint>
+  <link name="laser_sensor_link">
+          <inertial>
+                  <mass value="1e-5"/>
+                  <origin xyz="0 0 0" rpy="0 0 0"/>
+                  <inertia ixx="1e-6" ixy="0" ixz="0" iyy="1e-6" iyz="0" izz="1e-6"/>
+          </inertial>
+          <collision>
+                  <origin xyz="0 0 0" rpy="0 0 0"/>
+                  <geometry>
+                          <box size="0.1 0.1 0.1"/>
+                  </geometry>
+          </collision>
+          <visual>
+                  <origin xyz="0 0 0" rpy="0 0 0"/>
+                  <geometry>
+                          <cylinder radius="0.05" length="0.2"/>
+                  </geometry>
+          </visual>
+  </link> -->
   <!-- Colour -->
   <gazebo reference="base_link">
     <material>Gazebo/Green</material>
   </gazebo>
+<!--   <gazebo reference="laser_sensor_link">
+    <sensor type="ray" name="head_hokuyo_sensor">
+      <pose>0 0 0 0 0 0</pose>
+      <visualize>false</visualize>
+      <update_rate>40</update_rate>
+      <ray>
+        <scan>
+          <horizontal>
+            <samples>720</samples>
+            <resolution>1</resolution>
+            <min_angle>-1.570796</min_angle>
+            <max_angle>1.570796</max_angle>
+          </horizontal>
+        </scan>
+        <range>
+          <min>0.10</min>
+          <max>30.0</max>
+          <resolution>0.01</resolution>
+        </range>
+        <noise>
+          <type>gaussian</type>
+          <mean>0.0</mean>
+          <stddev>0.01</stddev>
+        </noise>
+      </ray>
+      <plugin name="gazebo_ros_head_hokuyo_controller" filename="libgazebo_ros_laser.so">
+        <topicName>/steer_bot/laser/scan</topicName>
+        <frameName>laser_sensor_link</frameName>
+      </plugin>
+    </sensor>
+  </gazebo> -->
 </robot>

File: steer_bot_description/urdf/wheel.xacro (robot description, xacro)
@@ -49,5 +49,5 @@
       <parent link="${parent}_link"/>
       <child link="${name}_steer_link"/>
-      <origin xyz="${base_length/2-axle_offset} 0 ${steer_height}" rpy="0 0 0"/>
+      <origin xyz="0 0 ${steer_height}" rpy="0 0 0"/>
       <axis xyz="0 0 1"/>
       <limit effort="${steer_effort}"

Commit message: added move_base components

File: steer_bot_description/urdf/steer_bot.urdf.xacro (robot description, xacro)
@@ -134,5 +134,5 @@
     <origin xyz="${-base_length/2+axle_offset} ${+base_width/2+axle_offset} 0" rpy="${-90 * deg_to_rad} 0 0"/>
   </xacro:rear_wheel_lr>
-<!--   <joint name="laser_sensor_joint" type="fixed">
+  <joint name="laser_sensor_joint" type="fixed">
       <origin xyz="0.2 0.0 ${base_height}" rpy="0 0 0"/>
       <parent link="base_link"/>
@@ -157,10 +157,10 @@
                   </geometry>
           </visual>
-  </link> -->
+  </link>
   <!-- Colour -->
   <gazebo reference="base_link">
     <material>Gazebo/Green</material>
   </gazebo>
-<!--   <gazebo reference="laser_sensor_link">
+  <gazebo reference="laser_sensor_link">
     <sensor type="ray" name="head_hokuyo_sensor">
       <pose>0 0 0 0 0 0</pose>
@@ -192,4 +192,4 @@
       </plugin>
     </sensor>
-  </gazebo> -->
+  </gazebo>
 </robot>

Commit message: wrapped up move_base files, workaround odometry from gazebo groundtruth pose, rviz visualization for navigation

File: steer_bot_description/urdf/steer_bot.urdf.xacro (robot description, xacro)
@@ -135,26 +135,26 @@
   </xacro:rear_wheel_lr>
   <joint name="laser_sensor_joint" type="fixed">
-      <origin xyz="0.2 0.0 ${base_height}" rpy="0 0 0"/>
-      <parent link="base_link"/>
-      <child link="laser_sensor_link"/>
+    <origin xyz="0.2 0.0 ${base_height}" rpy="0 0 0"/>
+    <parent link="base_link"/>
+    <child link="laser_sensor_link"/>
   </joint>
   <link name="laser_sensor_link">
-          <inertial>
-                  <mass value="1e-5"/>
-                  <origin xyz="0 0 0" rpy="0 0 0"/>
-                  <inertia ixx="1e-6" ixy="0" ixz="0" iyy="1e-6" iyz="0" izz="1e-6"/>
-          </inertial>
-          <collision>
-                  <origin xyz="0 0 0" rpy="0 0 0"/>
-                  <geometry>
-                          <box size="0.1 0.1 0.1"/>
-                  </geometry>
-          </collision>
-          <visual>
-                  <origin xyz="0 0 0" rpy="0 0 0"/>
-                  <geometry>
-                          <cylinder radius="0.05" length="0.2"/>
-                  </geometry>
-          </visual>
+    <inertial>
+      <mass value="1e-5"/>
+      <origin xyz="0 0 0" rpy="0 0 0"/>
+      <inertia ixx="1e-6" ixy="0" ixz="0" iyy="1e-6" iyz="0" izz="1e-6"/>
+    </inertial>
+    <collision>
+      <origin xyz="0 0 0" rpy="0 0 0"/>
+      <geometry>
+              <box size="0.1 0.1 0.1"/>
+      </geometry>
+    </collision>
+    <visual>
+      <origin xyz="0 0 0" rpy="0 0 0"/>
+      <geometry>
+              <cylinder radius="0.05" length="0.2"/>
+      </geometry>
+    </visual>
   </link>
   <!-- Colour -->
